Commit message: Created core URDF

File: description/robot.urdf.xacro (robot description, xacro)
@@ -2,3 +2,4 @@
 <robot xmlns:xacro="http://www.ros.org/wiki/xacro"  name="robot">
     <xacro:include filename="robot_core.xacro" />
+    <!--xacro:include filename="gazebo_control.xacro"/-->
 </robot>

File: description/robot_core.xacro (robot description, xacro)
@@ -19,88 +19,90 @@
         <parent link="base_link"/>
         <child link="chassis"/>
-        <origin xyz="-0.1 0 0"/>
+        <origin xyz="0 0 0.034"/>
     </joint>
     <link name="chassis">
         <visual>
-            <origin xyz="0.15 0 0.075"/>
+            <origin xyz="0.09 0 0.02" rpy="0 0 0"/>
             <geometry>
-                <box size="0.3 0.3 0.15"/>
+                <box size="0.23 0.215 0.040"/>
             </geometry>
             <material name="white"/>
         </visual>
         <collision>
-            <origin xyz="0.15 0 0.075"/>
+            <origin xyz="0.09 0 0.02" rpy="0 0 0"/>
             <geometry>
-                <box size="0.3 0.3 0.15"/>
+                <box size="0.23 0.215 0.040"/>
             </geometry>
         </collision>
         <xacro:inertial_box mass="0.5" x="0.3" y="0.3" z="0.15">
-            <origin xyz="0.15 0 0.075" rpy="0 0 0"/>
+            <origin xyz="-0.09 0 0.02" rpy="0 0 0"/>
         </xacro:inertial_box>
     </link>
-    <!-- LEFT WHEEL LINK-->
-    <joint name="left_wheel_joint" type="continuous">
+    <!--WHEELS-->
+    <!--Left-->
+     <joint name="wheel_joint_l" type="continuous">
         <parent link="base_link"/>
-        <child link="left_wheel"/>
-        <origin xyz="0 0.175 0" rpy="-${pi/2} 0 0"/>
+        <child link="wheel_l"/>
+        <origin xyz="-0.022 0.1205 0.034" rpy="-${pi/2} 0 0"/>
         <axis xyz="0 0 1"/>
     </joint>
-    <link name="left_wheel">
+    <link name="wheel_l">
         <visual>
             <geometry>
-                <cylinder radius="0.05" length="0.04"/>
+                <cylinder length="0.026" radius="0.034"/>
             </geometry>
+            <material name="orange"/>
         </visual>
         <collision>
             <geometry>
-                <cylinder radius="0.05" length="0.04"/>
+                <cylinder length="0.026" radius="0.034"/>
             </geometry>
         </collision>
-        <xacro:inertial_cylinder mass="0.1" length="0.04" radius="0.05">
-            <origin xyz ="0 0 0" rpy="0 0 0"/>
+        <xacro:inertial_cylinder mass="0.05" length="0.026" radius="0.034">
+            <origin xyz="0 0 0" rpy="0 0 0"/>
         </xacro:inertial_cylinder>
     </link>
-    <!-- RIGHT WHEEL LINK-->
-    <joint name="right_wheel_joint" type="continuous">
+    <!--Left-->
+     <joint name="wheel_joint_r" type="continuous">
         <parent link="base_link"/>
-        <child link="right_wheel"/>
-        <origin xyz="0 -0.175 0" rpy="${pi/2} 0 0"/>
+        <child link="wheel_r"/>
+        <origin xyz="-0.022 -0.1205 0.034" rpy="${pi/2} 0 0"/>
         <axis xyz="0 0 -1"/>
     </joint>
-    <link name="right_wheel">
+    <link name="wheel_r">
         <visual>
             <geometry>
-                <cylinder radius="0.05" length="0.04"/>
+                <cylinder length="0.026" radius="0.034"/>
             </geometry>
+            <material name="orange"/>
         </visual>
         <collision>
             <geometry>
-                <cylinder radius="0.05" length="0.04"/>
+                <cylinder length="0.026" radius="0.034"/>
             </geometry>
         </collision>
-        <xacro:inertial_cylinder mass="0.1" length="0.04" radius="0.05">
-            <origin xyz ="0 0 0" rpy="0 0 0"/>
+        <xacro:inertial_cylinder mass="0.05" length="0.026" radius="0.034">
+            <origin xyz="0 0 0" rpy="0 0 0"/>
         </xacro:inertial_cylinder>
     </link>
-    <!-- CASTER WHEEL LINK-->
-    <joint name="caster_wheel_joint" type="fixed">
+    <!-- BALL JOINT-->
+    <joint name="ball_joint" type="fixed">
         <parent link="chassis"/>
-        <child link="caster_wheel"/>
-        <origin xyz="0.24 0 0"/>
+        <child link="ball"/>
+        <origin xyz="0.145 0 0"/>
     </joint>
-    <link name="caster_wheel">
+    <link name="ball">
         <visual>
             <geometry>
-                <sphere radius="0.05"/>
+                <sphere radius="0.036"/>
             </geometry>
+            <material name="black"/>
         </visual>
         <collision>
             <geometry>
-                <sphere radius="0.05"/>
+                <sphere radius="0.036"/>
             </geometry>
+            <material name="black"/>
         </collision>
-        <xacro:inertial_sphere mass="0.1" radius="0.05">
-            <origin xyz="0 0 0" rpy="0 0 0"/>
-        </xacro:inertial_sphere>
     </link>
 </robot>
