Commit message: Committer: David <david@UbuntuRos.myguest.virtualbox.org>
 On branch main
 Your branch is ahead of 'origin/main' by 2 commits.
   (use "git push" to publish your local commits)

 Changes to be committed:
	deleted:    description/DiffRobotdae.dae
	deleted:    description/MainBody - Part 1.stl
	deleted:    description/Part 1.dae
	modified:   description/gazebo_control.xacro
	new file:   description/lidar.xacro
	modified:   description/robot.urdf.xacro
	modified:   description/robot_core.xacro

File: description/gazebo_control.xacro (robot description, xacro)
@@ -3,8 +3,8 @@
     <gazebo>
         <plugin name="diff_drive" filename="libgazebo_ros_diff_drive.so">
-            <left_joint>left_wheel_joint</left_joint>
-            <right_joint>right_wheel_joint</right_joint>
-            <wheel_separation>0.35</wheel_seperation>
-            <wheel_diameter>0.1</wheel_diameter>
+            <left_joint>wheel_joint_l</left_joint>
+            <right_joint>wheel_joint_r</right_joint>
+            <wheel_separation>0.241</wheel_separation>
+            <wheel_diameter>0.068</wheel_diameter>
             <!--limits-->
             <max_wheel_torque>200</max_wheel_torque>

File: description/robot.urdf.xacro (robot description, xacro)
@@ -2,4 +2,5 @@
 <robot xmlns:xacro="http://www.ros.org/wiki/xacro"  name="robot">
     <xacro:include filename="robot_core.xacro" />
-    <!--xacro:include filename="gazebo_control.xacro"/-->
+    <xacro:include filename="gazebo_control.xacro" />
+    <xacro:include filename="lidar.xacro" />
 </robot>

File: description/robot_core.xacro (robot description, xacro)
@@ -25,5 +25,5 @@
             <origin xyz="0.09 0 0.02" rpy="0 0 0"/>
             <geometry>
-                <box size="0.23 0.215 0.040"/>
+                <box size="0.23 0.214 0.040"/>
             </geometry>
             <material name="white"/>
@@ -32,9 +32,9 @@
             <origin xyz="0.09 0 0.02" rpy="0 0 0"/>
             <geometry>
-                <box size="0.23 0.215 0.040"/>
+                <box size="0.23 0.214 0.040"/>
             </geometry>
         </collision>
-        <xacro:inertial_box mass="0.5" x="0.3" y="0.3" z="0.15">
-            <origin xyz="-0.09 0 0.02" rpy="0 0 0"/>
+        <xacro:inertial_box mass="0.5" x="0.23" y="0.214" z="0.04">
+            <origin xyz="0.09 0 0.02" rpy="0 0 0"/>
         </xacro:inertial_box>
     </link>
@@ -95,5 +95,5 @@
         <visual>
             <geometry>
-                <sphere radius="0.036"/>
+                <sphere radius="0.034"/>
             </geometry>
             <material name="black"/>
@@ -101,8 +101,15 @@
         <collision>
             <geometry>
-                <sphere radius="0.036"/>
+                <sphere radius="0.034"/>
             </geometry>
             <material name="black"/>
         </collision>
+        <xacro:inertial_sphere mass="0.1" radius="0.034">
+            <origin xyz="0 0 0" rpy="0 0 0"/>
+        </xacro:inertial_sphere>
     </link>
+    <gazebo reference="ball">
+        <mu1 value="0.001"/>
+        <mu2 value="0.001"/>
+    </gazebo>
 </robot>
